File: can-transceiver.kicad_sch (KiCad schematic)
At the start: 18 parts, among them U8 ISOW1044

Commit message: Update tolerances, finish BOM
Parts:
- C31, C32: footprint Capacitor_SMD:C_0603_1608Metric -> Capacitor_SMD:C_1206_3216Metric
Changed lines of the file:
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@@
       (effects (font (size 1.27 1.27)) (justify left))
     )
-    (property "Footprint" "Capacitor_SMD:C_0603_1608Metric" (id 2) (at 81.28 48.26 0)
+    (property "Footprint" "Capacitor_SMD:C_1206_3216Metric" (id 2) (at 81.28 48.26 0)
       (effects (font (size 1.27 1.27)) hide)
     )
@@
       (effects (font (size 1.27 1.27)) (justify left))
     )
-    (property "Footprint" "Capacitor_SMD:C_0603_1608Metric" (id 2) (at 81.28 68.58 0)
+    (property "Footprint" "Capacitor_SMD:C_1206_3216Metric" (id 2) (at 81.28 68.58 0)
       (effects (font (size 1.27 1.27)) hide)
     )
